Commit message: Update code

File: urdf/omni_robot.xacro (robot description, xacro)
@@ -1,5 +1,5 @@
 <?xml version='1.0'?>
 <robot name="omni_robot" xmlns:xacro="http://www.ros.org/wiki/xacro">
-  	<xacro:include filename="$(find omni_gazebo)/urdf/omni_robot.gazebo" />
+  	<xacro:include filename="$(find omni_learning)/urdf/omni_robot.gazebo" />
 	<xacro:property name="scale" value="0.01" />
   	<link name="base_footprint"></link>
@@ -94,5 +94,5 @@
 			<origin xyz="-0.01 0 -0.03" rpy="1.5707 0 1.5707"/>
 			<geometry>
-				<mesh filename="package://omni_gazebo/meshes/astra.dae" scale="0.001 0.001 0.001" />
+				<mesh filename="package://omni_learning/meshes/astra.dae" scale="0.001 0.001 0.001" />
 			</geometry>
 		</visual>
@@ -128,5 +128,5 @@
 			<origin xyz="0 0 0" rpy="1.5707 0 3.1412"/>
 			<geometry>
-				<mesh filename="package://omni_gazebo/meshes/rplidar.dae" scale="0.001 0.001 0.001" />
+				<mesh filename="package://omni_learning/meshes/rplidar.dae" scale="0.001 0.001 0.001" />
 			</geometry>
 		</collision>
@@ -134,5 +134,5 @@
 			<origin xyz="0 0 0" rpy="1.5707 0 4.71"/>
 			<geometry>
-				<mesh filename="package://omni_gazebo/meshes/rplidar.dae" scale="0.001 0.001 0.001" />
+				<mesh filename="package://omni_learning/meshes/rplidar.dae" scale="0.001 0.001 0.001" />
 			</geometry>
 		</visual>
@@ -193,5 +193,5 @@
 			<origin xyz="0 0 0" rpy="0 0 0.0" />
 			<geometry>
-				<mesh filename="package://omni_gazebo/meshes/rim.stl" scale="5 5 5"/>
+				<mesh filename="package://omni_learning/meshes/rim.stl" scale="5 5 5"/>
 			</geometry>
 			<material name="left_rim_material">
@@ -202,5 +202,5 @@
 		<collision>
 			<geometry>
-				<mesh filename="package://omni_gazebo/meshes/rim.stl" scale="5 5 5"/>
+				<mesh filename="package://omni_learning/meshes/rim.stl" scale="5 5 5"/>
 			</geometry>
 		</collision>
@@ -233,5 +233,5 @@
 		<origin xyz="0 0 0" rpy="0 0 0.0" />
 		<geometry>
-			<mesh filename="package://omni_gazebo/meshes/rim.stl" scale="5 5 5"/>
+			<mesh filename="package://omni_learning/meshes/rim.stl" scale="5 5 5"/>
 		</geometry>
 		<material name="left_rim_material">
@@ -242,5 +242,5 @@
 		<collision>
 			<geometry>
-				<mesh filename="package://omni_gazebo/meshes/rim.stl" scale="5 5 5"/>
+				<mesh filename="package://omni_learning/meshes/rim.stl" scale="5 5 5"/>
 			</geometry>
 		</collision>
@@ -273,5 +273,5 @@
 		<origin xyz="0 0 0" rpy="0 0 0.0" />
 		<geometry>
-			<mesh filename="package://omni_gazebo/meshes/rim.stl" scale="5 5 5"/>
+			<mesh filename="package://omni_learning/meshes/rim.stl" scale="5 5 5"/>
 		</geometry>
 			<material name="left_rim_material">
@@ -282,5 +282,5 @@
 		<collision>
 			<geometry>
-				<mesh filename="package://omni_gazebo/meshes/rim.stl" scale="5 5 5"/>
+				<mesh filename="package://omni_learning/meshes/rim.stl" scale="5 5 5"/>
 			</geometry>
 		</collision>
@@ -297,5 +297,5 @@
 			<origin xyz="0 0 0" rpy="0 0 0"/>
 			<geometry>
-				<mesh filename="package://omni_gazebo/meshes/roller.stl" scale="5 5 5"/>
+				<mesh filename="package://omni_learning/meshes/roller.stl" scale="5 5 5"/>
 			</geometry>
 			<material name="bottem_left_roller_e_material">
@@ -316,5 +316,5 @@
 		<collision>
 			<geometry>
-				<mesh filename="package://omni_gazebo/meshes/roller.stl" scale="5 5 5"/>
+				<mesh filename="package://omni_learning/meshes/roller.stl" scale="5 5 5"/>
 			</geometry>
 		</collision>
@@ -346,5 +346,5 @@
 		<visual>
 			<geometry>
-				<mesh filename="package://omni_gazebo/meshes/roller.stl" scale="5 5 5"/>
+				<mesh filename="package://omni_learning/meshes/roller.stl" scale="5 5 5"/>
 			</geometry>
 			<material name="bottem_left_roller_e_material">
@@ -354,5 +354,5 @@
 		<collision>
 			<geometry>
-				<mesh filename="package://omni_gazebo/meshes/roller.stl" scale="5 5 5"/>
+				<mesh filename="package://omni_learning/meshes/roller.stl" scale="5 5 5"/>
 			</geometry>
 		</collision>
@@ -384,5 +384,5 @@
 		<visual>
 			<geometry>
-				<mesh filename="package://omni_gazebo/meshes/roller.stl" scale="5 5 5"/>
+				<mesh filename="package://omni_learning/meshes/roller.stl" scale="5 5 5"/>
 			</geometry>
 			<material name="bottem_left_roller_n_material">
@@ -392,5 +392,5 @@
 		<collision>
 			<geometry>
-				<mesh filename="package://omni_gazebo/meshes/roller.stl" scale="5 5 5"/>
+				<mesh filename="package://omni_learning/meshes/roller.stl" scale="5 5 5"/>
 			</geometry>
 		</collision>
@@ -419,5 +419,5 @@
 		<visual>
 			<geometry>
-				<mesh filename="package://omni_gazebo/meshes/roller.stl" scale="5 5 5"/>
+				<mesh filename="package://omni_learning/meshes/roller.stl" scale="5 5 5"/>
 			</geometry>
 			<material name="bottem_left_roller_nw_material">
@@ -427,5 +427,5 @@
 		<collision>
 			<geometry>
-				<mesh filename="package://omni_gazebo/meshes/roller.stl" scale="5 5 5"/>
+				<mesh filename="package://omni_learning/meshes/roller.stl" scale="5 5 5"/>
 			</geometry>
 		</collision>
@@ -454,5 +454,5 @@
 		<visual>
 			<geometry>
-				<mesh filename="package://omni_gazebo/meshes/roller.stl" scale="5 5 5"/>
+				<mesh filename="package://omni_learning/meshes/roller.stl" scale="5 5 5"/>
 			</geometry>
 			<material name="bottem_left_roller_w_material">
@@ -462,5 +462,5 @@
 		<collision>
 			<geometry>
-				<mesh filename="package://omni_gazebo/meshes/roller.stl" scale="5 5 5"/>
+				<mesh filename="package://omni_learning/meshes/roller.stl" scale="5 5 5"/>
 			</geometry>
 		</collision>
@@ -489,5 +489,5 @@
 		<visual>
 			<geometry>
-				<mesh filename="package://omni_gazebo/meshes/roller.stl" scale="5 5 5"/>
+				<mesh filename="package://omni_learning/meshes/roller.stl" scale="5 5 5"/>
 			</geometry>
 			<material name="bottem_left_roller_sw_material">
@@ -497,5 +497,5 @@
 		<collision>
 			<geometry>
-				<mesh filename="package://omni_gazebo/meshes/roller.stl" scale="5 5 5"/>
+				<mesh filename="package://omni_learning/meshes/roller.stl" scale="5 5 5"/>
 			</geometry>
 		</collision>
@@ -524,5 +524,5 @@
 		<visual>
 			<geometry>
-				<mesh filename="package://omni_gazebo/meshes/roller.stl" scale="5 5 5"/>
+				<mesh filename="package://omni_learning/meshes/roller.stl" scale="5 5 5"/>
 			</geometry>
 			<material name="bottem_left_roller_s_material">
@@ -532,5 +532,5 @@
 		<collision>
 			<geometry>
-				<mesh filename="package://omni_gazebo/meshes/roller.stl" scale="5 5 5"/>
+				<mesh filename="package://omni_learning/meshes/roller.stl" scale="5 5 5"/>
 			</geometry>
 		</collision>
@@ -559,5 +559,5 @@
 		<visual>
 			<geometry>
-				<mesh filename="package://omni_gazebo/meshes/roller.stl" scale="5 5 5"/>
+				<mesh filename="package://omni_learning/meshes/roller.stl" scale="5 5 5"/>
 			</geometry>
 			<material name="bottem_left_roller_se_material">
@@ -567,5 +567,5 @@
 		<collision>
 			<geometry>
-				<mesh filename="package://omni_gazebo/meshes/roller.stl" scale="5 5 5"/>
+				<mesh filename="package://omni_learning/meshes/roller.stl" scale="5 5 5"/>
 			</geometry>
 		</collision>
@@ -584,5 +584,5 @@
 			<origin xyz="0 0 0"	rpy="0 0 0"/>
 			<geometry>
-				<mesh filename="package://omni_gazebo/meshes/roller.stl" scale="5 5 5"/>
+				<mesh filename="package://omni_learning/meshes/roller.stl" scale="5 5 5"/>
 			</geometry>
 			<material name="bottem_right_roller_e_material">
@@ -603,5 +603,5 @@
 		<collision>
 			<geometry>
-				<mesh filename="package://omni_gazebo/meshes/roller.stl" scale="5 5 5"/>
+				<mesh filename="package://omni_learning/meshes/roller.stl" scale="5 5 5"/>
 			</geometry>
 		</collision>
@@ -630,5 +630,5 @@
 		<visual>
 			<geometry>
-				<mesh filename="package://omni_gazebo/meshes/roller.stl" scale="5 5 5"/>
+				<mesh filename="package://omni_learning/meshes/roller.stl" scale="5 5 5"/>
 			</geometry>
 			<material name="bottem_right_roller_e_material">
@@ -638,5 +638,5 @@
 		<collision>
 			<geometry>
-				<mesh filename="package://omni_gazebo/meshes/roller.stl" scale="5 5 5"/>
+				<mesh filename="package://omni_learning/meshes/roller.stl" scale="5 5 5"/>
 			</geometry>
 		</collision>
@@ -665,5 +665,5 @@
 		<visual>
 			<geometry>
-				<mesh filename="package://omni_gazebo/meshes/roller.stl" scale="5 5 5"/>
+				<mesh filename="package://omni_learning/meshes/roller.stl" scale="5 5 5"/>
 			</geometry>
 			<material name="bottem_right_roller_n_material">
@@ -673,5 +673,5 @@
 		<collision>
 			<geometry>
-				<mesh filename="package://omni_gazebo/meshes/roller.stl" scale="5 5 5"/>
+				<mesh filename="package://omni_learning/meshes/roller.stl" scale="5 5 5"/>
 			</geometry>
 		</collision>
@@ -700,5 +700,5 @@
 		<visual>
 			<geometry>
-				<mesh filename="package://omni_gazebo/meshes/roller.stl" scale="5 5 5"/>
+				<mesh filename="package://omni_learning/meshes/roller.stl" scale="5 5 5"/>
 			</geometry>
 			<material name="bottem_right_roller_nw_material">
@@ -708,5 +708,5 @@
 		<collision>
 			<geometry>
-				<mesh filename="package://omni_gazebo/meshes/roller.stl" scale="5 5 5"/>
+				<mesh filename="package://omni_learning/meshes/roller.stl" scale="5 5 5"/>
 			</geometry>
 		</collision>
@@ -735,5 +735,5 @@
 		<visual>
 			<geometry>
-				<mesh filename="package://omni_gazebo/meshes/roller.stl" scale="5 5 5"/>
+				<mesh filename="package://omni_learning/meshes/roller.stl" scale="5 5 5"/>
 			</geometry>
 			<material name="bottem_right_roller_w_material">
@@ -743,5 +743,5 @@
 		<collision>
 			<geometry>
-				<mesh filename="package://omni_gazebo/meshes/roller.stl" scale="5 5 5"/>
+				<mesh filename="package://omni_learning/meshes/roller.stl" scale="5 5 5"/>
 			</geometry>
 		</collision>
@@ -770,5 +770,5 @@
 		<visual>
 			<geometry>
-				<mesh filename="package://omni_gazebo/meshes/roller.stl" scale="5 5 5"/>
+				<mesh filename="package://omni_learning/meshes/roller.stl" scale="5 5 5"/>
 			</geometry>
 			<material name="bottem_right_roller_sw_material">
@@ -778,5 +778,5 @@
 		<collision>
 			<geometry>
-				<mesh filename="package://omni_gazebo/meshes/roller.stl" scale="5 5 5"/>
+				<mesh filename="package://omni_learning/meshes/roller.stl" scale="5 5 5"/>
 			</geometry>
 		</collision>
@@ -805,5 +805,5 @@
 		<visual>
 			<geometry>
-				<mesh filename="package://omni_gazebo/meshes/roller.stl" scale="5 5 5"/>
+				<mesh filename="package://omni_learning/meshes/roller.stl" scale="5 5 5"/>
 			</geometry>
 			<material name="bottem_right_roller_s_material">
@@ -813,5 +813,5 @@
 		<collision>
 			<geometry>
-				<mesh filename="package://omni_gazebo/meshes/roller.stl" scale="5 5 5"/>
+				<mesh filename="package://omni_learning/meshes/roller.stl" scale="5 5 5"/>
 			</geometry>
 		</collision>
@@ -840,5 +840,5 @@
 		<visual>
 			<geometry>
-				<mesh filename="package://omni_gazebo/meshes/roller.stl" scale="5 5 5"/>
+				<mesh filename="package://omni_learning/meshes/roller.stl" scale="5 5 5"/>
 			</geometry>
 			<material name="bottem_right_roller_se_material">
@@ -848,5 +848,5 @@
 		<collision>
 			<geometry>
-				<mesh filename="package://omni_gazebo/meshes/roller.stl" scale="5 5 5"/>
+				<mesh filename="package://omni_learning/meshes/roller.stl" scale="5 5 5"/>
 			</geometry>
 		</collision>
@@ -865,5 +865,5 @@
 			<origin	xyz="0 0 0"	rpy="0 0 0"/>
 			<geometry>
-				<mesh filename="package://omni_gazebo/meshes/roller.stl" scale="5 5 5"/>
+				<mesh filename="package://omni_learning/meshes/roller.stl" scale="5 5 5"/>
 			</geometry>
 			<material name="right_left_roller_e_material">
@@ -884,5 +884,5 @@
 		<collision>
 			<geometry>
-				<mesh filename="package://omni_gazebo/meshes/roller.stl" scale="5 5 5"/>
+				<mesh filename="package://omni_learning/meshes/roller.stl" scale="5 5 5"/>
 			</geometry>
 		</collision>
@@ -911,5 +911,5 @@
 		<visual>
 			<geometry>
-				<mesh filename="package://omni_gazebo/meshes/roller.stl" scale="5 5 5"/>
+				<mesh filename="package://omni_learning/meshes/roller.stl" scale="5 5 5"/>
 			</geometry>
 			<material name="right_left_roller_e_material">
@@ -919,5 +919,5 @@
 		<collision>
 			<geometry>
-				<mesh filename="package://omni_gazebo/meshes/roller.stl" scale="5 5 5"/>
+				<mesh filename="package://omni_learning/meshes/roller.stl" scale="5 5 5"/>
 			</geometry>
 		</collision>
@@ -946,5 +946,5 @@
 		<visual>
 			<geometry>
-				<mesh filename="package://omni_gazebo/meshes/roller.stl" scale="5 5 5"/>
+				<mesh filename="package://omni_learning/meshes/roller.stl" scale="5 5 5"/>
 			</geometry>
 			<material name="right_left_roller_n_material">
@@ -954,5 +954,5 @@
 		<collision>
 			<geometry>
-				<mesh filename="package://omni_gazebo/meshes/roller.stl" scale="5 5 5"/>
+				<mesh filename="package://omni_learning/meshes/roller.stl" scale="5 5 5"/>
 			</geometry>
 		</collision>
@@ -981,5 +981,5 @@
 		<visual>
 			<geometry>
-				<mesh filename="package://omni_gazebo/meshes/roller.stl" scale="5 5 5"/>
+				<mesh filename="package://omni_learning/meshes/roller.stl" scale="5 5 5"/>
 			</geometry>
 			<material name="right_left_roller_nw_material">
@@ -989,5 +989,5 @@
 		<collision>
 			<geometry>
-				<mesh filename="package://omni_gazebo/meshes/roller.stl" scale="5 5 5"/>
+				<mesh filename="package://omni_learning/meshes/roller.stl" scale="5 5 5"/>
 			</geometry>
 		</collision>
@@ -1016,5 +1016,5 @@
 		<visual>
 			<geometry>
-				<mesh filename="package://omni_gazebo/meshes/roller.stl" scale="5 5 5"/>
+				<mesh filename="package://omni_learning/meshes/roller.stl" scale="5 5 5"/>
 			</geometry>
 			<material name="right_left_roller_w_material">
@@ -1024,5 +1024,5 @@
 		<collision>
 			<geometry>
-				<mesh filename="package://omni_gazebo/meshes/roller.stl" scale="5 5 5"/>
+				<mesh filename="package://omni_learning/meshes/roller.stl" scale="5 5 5"/>
 			</geometry>
 		</collision>
@@ -1051,5 +1051,5 @@
 		<visual>
 			<geometry>
-				<mesh filename="package://omni_gazebo/meshes/roller.stl" scale="5 5 5"/>
+				<mesh filename="package://omni_learning/meshes/roller.stl" scale="5 5 5"/>
 			</geometry>
 			<material name="right_left_roller_sw_material">
@@ -1059,5 +1059,5 @@
 		<collision>
 			<geometry>
-				<mesh filename="package://omni_gazebo/meshes/roller.stl" scale="5 5 5"/>
+				<mesh filename="package://omni_learning/meshes/roller.stl" scale="5 5 5"/>
 			</geometry>
 		</collision>
@@ -1086,5 +1086,5 @@
 		<visual>
 			<geometry>
-				<mesh filename="package://omni_gazebo/meshes/roller.stl" scale="5 5 5"/>
+				<mesh filename="package://omni_learning/meshes/roller.stl" scale="5 5 5"/>
 			</geometry>
 			<material name="right_left_roller_s_material">
@@ -1094,5 +1094,5 @@
 		<collision>
 			<geometry>
-				<mesh filename="package://omni_gazebo/meshes/roller.stl" scale="5 5 5"/>
+				<mesh filename="package://omni_learning/meshes/roller.stl" scale="5 5 5"/>
 			</geometry>
 		</collision>
@@ -1121,5 +1121,5 @@
 		<visual>
 			<geometry>
-				<mesh filename="package://omni_gazebo/meshes/roller.stl" scale="5 5 5"/>
+				<mesh filename="package://omni_learning/meshes/roller.stl" scale="5 5 5"/>
 			</geometry>
 			<material name="right_left_roller_se_material">
@@ -1129,5 +1129,5 @@
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